Commit message: added acceleration from file

File: arctos_description/urdf/arctos.xacro (robot description, xacro)
@@ -7,4 +7,5 @@
   <xacro:arg name="abs_motion" default="true" />
   <xacro:arg name="initial_positions_file" default="$(find arctos_description)/config/initial_positions.yaml" />
+  <xacro:arg name="joint_limits_file" default="$(find arctos_description)/config/joint_limits.yaml" />
   <xacro:include filename="$(find arctos_description)/urdf/materials.xacro" />
   <xacro:include filename="$(find arctos_description)/urdf/joint_link.xacro" />

File: arctos_description/urdf/arctos_base.xacro (robot description, xacro)
@@ -1,5 +1,7 @@
 <?xml version="1.0"?>
 <robot xmlns:xacro="http://www.ros.org/wiki/xacro">
-  <xacro:include filename="$(find arctos_description)/urdf/joint_link.xacro" />
+    <xacro:include filename="$(find arctos_description)/urdf/joint_link.xacro" />
+    <xacro:property name="joint_limits"
+        value="${xacro.load_yaml(joint_limits_file)['joint_limits']}" />
     <link name="world" />
     <xacro:arctos_link
@@ -83,5 +85,7 @@
         origin_xyz="0.0 0.000529 0.111" origin_rpy="0 0 0"
         axis_xyz="0 0 1"
-        limit_u="${2*pi}" limit_l="${-2*pi}" limit_e="100.0" limit_v="100.0"
+        limit_u="${2*pi}" limit_l="${-2*pi}" limit_e="100.0"
+        limit_v="${joint_limits['X_joint']['max_velocity']}"
+        limit_a="${joint_limits['X_joint']['max_acceleration']}"
     />
     <xacro:arctos_joint
@@ -90,5 +94,7 @@
         origin_xyz="-0.05713 -0.020885 0.178378" origin_rpy="0 0 0"
         axis_xyz="1 0 0"
-        limit_u="${2*pi}" limit_l="${-2*pi}" limit_e="100.0" limit_v="100.0"
+        limit_u="${2*pi}" limit_l="${-2*pi}" limit_e="100.0"
+        limit_v="${joint_limits['Y_joint']['max_velocity']}"
+        limit_a="${joint_limits['Y_joint']['max_acceleration']}"
     />
     <xacro:arctos_joint
@@ -97,5 +103,7 @@
         origin_xyz="0.10013 0.001311 0.261007" origin_rpy="0 0 0"
         axis_xyz="-1 0 0"
-        limit_u="${pi}" limit_l="${-pi}" limit_e="100.0" limit_v="100.0"
+        limit_u="${pi}" limit_l="${-pi}" limit_e="100.0"
+        limit_v="${joint_limits['Z_joint']['max_velocity']}"
+        limit_a="${joint_limits['Z_joint']['max_acceleration']}"
     />
     <xacro:arctos_joint
@@ -104,5 +112,7 @@
         origin_xyz="-0.042999 -0.139695 0.021705" origin_rpy="0 0 0"
         axis_xyz="0 1 0"
-        limit_u="${2*pi}" limit_l="${-2*pi}" limit_e="100.0" limit_v="100.0"
+        limit_u="${2*pi}" limit_l="${-2*pi}" limit_e="100.0"
+        limit_v="${joint_limits['A_joint']['max_velocity']}"
+        limit_a="${joint_limits['A_joint']['max_acceleration']}"
     />
     <xacro:arctos_joint
@@ -111,5 +121,7 @@
         origin_xyz="-0.039012 -0.121187 -0.001774" origin_rpy="0 0 0"
         axis_xyz="-1 0 0"
-        limit_u="${2*pi}" limit_l="${-2*pi}" limit_e="100.0" limit_v="100.0"
+        limit_u="${2*pi}" limit_l="${-2*pi}" limit_e="100.0"
+        limit_v="${joint_limits['B_joint']['max_velocity']}"
+        limit_a="${joint_limits['B_joint']['max_acceleration']}"
     />
     <xacro:arctos_joint
@@ -118,5 +130,7 @@
         origin_xyz="0.039204 -0.033835 0.0" origin_rpy="0 0 0"
         axis_xyz="0 1 0"
-        limit_u="${2*pi}" limit_l="${-2*pi}" limit_e="100.0" limit_v="100.0"
+        limit_u="${2*pi}" limit_l="${-2*pi}" limit_e="100.0"
+        limit_v="${joint_limits['C_joint']['max_velocity']}"
+        limit_a="${joint_limits['C_joint']['max_acceleration']}"
     />
 </robot>

File: arctos_description/urdf/arctos_gripper.xacro (robot description, xacro)
@@ -40,5 +40,7 @@
     <origin xyz="0.007741 -0.039998 0.029551" rpy="0 0 0" />
     <axis xyz="0 0 -1" />
-    <limit upper="0.015" lower="0.0" effort="100.0" velocity="100.0" />
+    <limit upper="0.015" lower="0.0" effort="100.0"
+      velocity="${joint_limits['Left_jaw_joint']['max_velocity']}"
+      acceleration="${joint_limits['Left_jaw_joint']['max_acceleration']}" />
     <dynamics damping="0.0" friction="0.0" />
   </joint>
@@ -48,5 +50,7 @@
     <origin xyz="0.007741 -0.039998 -0.030449" rpy="0 0 0" />
     <axis xyz="0 0 1" />
-    <limit upper="0.015" lower="0.0" effort="100.0" velocity="100.0" />
+    <limit upper="0.015" lower="0.0" effort="100.0"
+      velocity="${joint_limits['Right_jaw_joint']['max_velocity']}"
+      acceleration="${joint_limits['Right_jaw_joint']['max_acceleration']}" />
     <mimic joint="Left_jaw_joint" multiplier="1.0" offset="0.0" />
     <dynamics damping="0.0" friction="0.0" />

File: arctos_description/urdf/joint_link.xacro (robot description, xacro)
@@ -27,5 +27,5 @@
   <!-- Define arctos_joint macro with a default value for axis_xyz -->
   <xacro:macro name="arctos_joint"
-    params="name type parent child origin_xyz origin_rpy axis_xyz='0 0 0' limit_u limit_l limit_e limit_v">
+    params="name type parent child origin_xyz origin_rpy axis_xyz='0 0 0' limit_u limit_l limit_e limit_v limit_a">
     <joint name="${name}" type="${type}">
       <parent link="${parent}" />
@@ -33,5 +33,5 @@
       <origin xyz="${origin_xyz}" rpy="${origin_rpy}" />
       <axis xyz="${axis_xyz}" />
-      <limit upper="${limit_u}" lower="${limit_l}" effort="${limit_e}" velocity="${limit_v}" acceleration="0.0" />
+      <limit upper="${limit_u}" lower="${limit_l}" effort="${limit_e}" velocity="${limit_v}" acceleration="${limit_a}" />
     </joint>
   </xacro:macro>
