Commit message: fixed bug

File: arctos_description/urdf/arctos_base.xacro (robot description, xacro)
@@ -2,6 +2,6 @@
 <robot xmlns:xacro="http://www.ros.org/wiki/xacro">
     <xacro:include filename="$(find arctos_description)/urdf/joint_link.xacro" />
-    <xacro:property name="joint_limits"
-        value="${xacro.load_yaml(joint_limits_file)['joint_limits']}" />
+    <xacro:property name="joint_limits_path" value="$(arg joint_limits_file)" />
+    <xacro:property name="joint_limits" value="${xacro.load_yaml(joint_limits_path)['joint_limits']}" />
     <link name="world" />
     <xacro:arctos_link
